File: flex_mems/flex_aufsatz/flex_aufsatz.kicad_pcb (KiCad board)
At the start: 2 copper layers, 0 parts

Commit message: Schematics done
Parts:
- added C1: 100nF, Capacitor_SMD:C_0402_1005Metric, F.Cu at (114.2, 77.7)
- added C2: 100nF, Capacitor_SMD:C_0402_1005Metric, F.Cu at (114.2, 79.7)
- added C3: 2.2uF, Capacitor_SMD:C_0402_1005Metric, F.Cu at (114.2, 81.7)
- added C4: 2.2uF, Capacitor_SMD:C_0402_1005Metric, F.Cu at (114.2, 83.6)
- added C6: 2.2uF, Capacitor_SMD:C_0402_1005Metric, F.Cu at (114.2, 85.6)
- added IC1: ADPL44002AUJZ-1.8-R7, ADPL44002AUJZ-1.8:SOT95P280X100-5N, F.Cu at (115.4, 69.1)
- added J1: Conn_01x22_Socket, Connector_PinSocket_2.54mm:PinSocket_1x22_P2.54mm_Vertical, F.Cu at (105.9, 69.2)
- added J2: Conn_01x22_Socket, Connector_PinSocket_2.54mm:PinSocket_1x22_P2.54mm_Vertical, F.Cu at (110.5, 69.2)
- added J3: 10164228-0101A1RLF, header:AMPHENOL_10164228-0101A1RLF, B.Cu at (106.1, 63.9)
- added J4: 10164228-0101A1RLF, header:AMPHENOL_10164228-0101A1RLF, B.Cu at (111.2, 63.9)
- added U1: ADAU7118ACPZRL, mux:QFN50P300X300X80-17N-D, F.Cu at (115.4, 74.1)
