File: flex_mems/flex_mems.kicad_pcb (KiCad board)
At the start: 2 copper layers, 311.5 x 65 mm, 20 parts, among them J1 10164227-0101A1RLF, J2 10164227-0101A1RLF

Commit message: Schematics done
Parts:
- added C7: 2.2uF, Capacitor_SMD:C_0402_1005Metric, F.Cu at (269.0, 128.0)
- added C8: 2.2uF, Capacitor_SMD:C_0402_1005Metric, F.Cu at (381.5, 148.5)
Routing:
- net GNDR: track 413.6 -> 419.5 mm, vias 9 -> 10
- net GNDL: track 138.6 -> 141.0 mm
- net +3V3L: track 125.6 -> 127.6 mm
- net +3V3R: track 392.9 -> 394.2 mm
- net /MIC_CLK: track 482.1 -> 481.4 mm

Commit message: GND zone update
Parts:
- added C10: 2.2uF, Capacitor_SMD:C_0402_1005Metric, F.Cu at (136.9, 146.6)
- added C11: 2.2uF, Capacitor_SMD:C_0402_1005Metric, F.Cu at (223.5, 127.2)
- added C9: 2.2uF, Capacitor_SMD:C_0402_1005Metric, F.Cu at (308.7, 146.4)
Routing:
- net +3V3R: track 394.2 -> 404.3 mm, vias 9 -> 11
- net GNDR: track 419.5 -> 427.2 mm, vias 10 -> 13
- net +3V3L: track 127.6 -> 132.5 mm, vias 3 -> 4
- net GNDL: track 141.0 -> 145.5 mm, vias 5 -> 6
- net /MIC_DOUT_0: track 296.5 -> 297.4 mm
- net /MIC_DOUT_2: track 106.7 -> 107.5 mm
- net /MIC_DOUT_1: track 187.8 -> 188.4 mm
- added copper zone on B.Cu, net GNDL
- added copper zone on F.Cu, net GNDL
- added copper zone on B.Cu, net GNDR
- added copper zone on F.Cu, net GNDR
